Commit message: Planar movement

File: tolya_ws/src/tolya_description/urdf/base.xacro (robot description, xacro)
@@ -3,28 +3,65 @@
     <xacro:macro name="base">
         <link name='base_link'>
-        <inertial>
-            <mass value="0.05"/>
-            <origin xyz="0.0 0 0" rpy=" 0 0 0"/>
-            <inertia
-                ixx="0.1" ixy="0" ixz="0"
-                iyy="0.1" iyz="0"
-                izz="0.1"
-            />
-        </inertial>
-        <collision name='base_collision'>
-            <origin xyz="0 0 0.06" rpy="0 0 0"/>
-            <geometry>
-                <box size="0.15 0.257 0.1"/>
-            </geometry>
-        </collision>
-        <visual name='base_visual'>
-            <origin xyz="0 0 0.06" rpy="0 0 0"/>
-            <!-- <origin xyz="-0.187 0 0" rpy="0 0 ${pi}"/> -->
-            <geometry>
-                <box size="0.1 0.257 0.1"/>
-                <!-- <mesh scale="0.001 0.001 0.001" filename="$(find tolya_description)/meshes/base.stl"/> -->
-            </geometry>
-        </visual>
+            <inertial>
+                <mass value="0.05"/>
+                <origin xyz="0.0 0 0" rpy=" 0 0 0"/>
+                <inertia
+                    ixx="0.1" ixy="0" ixz="0"
+                    iyy="0.1" iyz="0"
+                    izz="0.1"
+                />
+            </inertial>
+            <collision name='base_collision'>
+                <origin xyz="0 0 0.06" rpy="0 0 0"/>
+                <geometry>
+                    <box size="0.15 0.257 0.1"/>
+                </geometry>
+            </collision>
+            <visual name='base_visual'>
+                <origin xyz="0 0 0.06" rpy="0 0 0"/>
+                <!-- <origin xyz="-0.187 0 0" rpy="0 0 ${pi}"/> -->
+                <geometry>
+                    <box size="0.1 0.257 0.1"/>
+                    <!-- <mesh scale="0.001 0.001 0.001" filename="$(find tolya_description)/meshes/base.stl"/> -->
+                </geometry>
+            </visual>
         </link>
+        <link name="base_footprint">
+            <visual name="base_footprint_visual">
+                <origin xyz="0 0 0" rpy="0 0 0" />
+                <geometry>
+                    <box size="0.001 0.001 0.001" />
+                </geometry>
+            </visual>
+            <inertial>
+                <mass value="0.05"/>
+                <origin xyz="0.0 0 0" rpy=" 0 0 0"/>
+                <inertia
+                    ixx="0" ixy="0" ixz="0"
+                    iyy="0" iyz="0"
+                    izz="0"
+                />
+            </inertial>
+            <collision name='base_footprint_collision'>
+                <origin xyz="0 0 0" rpy="0 0 0"/>
+                <geometry>
+                    <box size="0.001 0.001 0.001" />
+                </geometry>
+            </collision>
+        </link>
+        <joint name="base_link_joint" type="fixed">
+            <origin xyz="0 0 0.05" rpy="0 0 0" />
+            <parent link="base_footprint"/>
+            <child link="base_link" />
+        </joint>
+        <gazebo>
+            <plugin name="object_controller" filename="libgazebo_ros_planar_move.so">
+                <commandTopic>cmd_vel</commandTopic>
+                <odometryTopic>odom</odometryTopic>
+                <odometryFrame>odom</odometryFrame>
+                <odometryRate>20.0</odometryRate>
+                <robotBaseFrame>base_footprint</robotBaseFrame>
+            </plugin>
+        </gazebo>
     </xacro:macro>
 </robot>

File: tolya_ws/src/tolya_description/urdf/tolya.xacro (robot description, xacro)
@@ -3,4 +3,5 @@
   <xacro:include filename="base.xacro" />
   <xacro:include filename="wheel.xacro" />
+  <xacro:include filename="sensors.xacro" />
   <xacro:base/>
   <xacro:wheel parent="base_link" origin_xyz="0.065 0.059 0.03" number="1"/>
@@ -8,3 +9,4 @@
   <xacro:wheel parent="base_link" origin_xyz="0.065 -0.059 0.03" number="3"/>
   <xacro:wheel parent="base_link" origin_xyz="-0.065 0.059 0.03" number="4"/>
+  <xacro:sensors parent="base_link"/>
 </robot>

File: tolya_ws/src/tolya_description/urdf/wheel.xacro (robot description, xacro)
@@ -1,35 +1,34 @@
 <?xml version='1.0'?>
 <robot xmlns:xacro="http://www.ros.org/wiki/xacro">
-    <xacro:macro name="wheel"  params="origin_xyz number parent">
+    <xacro:macro name="wheel" params="origin_xyz number parent">
         <link name='wheel_link_${number}'>
-        <inertial>
-            <mass value="0.05"/>
-            <origin xyz="0 0 0" rpy=" 0 0 0"/>
-            <inertia
-                ixx="0.1" ixy="0" ixz="0"
-                iyy="0.1" iyz="0"
-                izz="0.1"
-            />
-        </inertial>
-        <collision name='wheel_collision_${number}'>
-            <origin xyz="0 0 0" rpy="0 0 0"/>
-            <geometry>
-                <cylinder radius="0.03" length="0.03"/>
-            </geometry>
-        </collision>
-        <visual name='wheel_visual_${number}'>
-            <origin xyz="0 0 0" rpy="0 0 0"/>
-            <geometry>
-                <!-- <mesh filename="$(find tolya_description)/meshes/wheel.stl"/> -->
-                <cylinder radius="0.03" length="0.03"/>
-            </geometry>
-        </visual>
+            <inertial>
+                <mass value="0.05"/>
+                <origin xyz="0 0 0" rpy=" 0 0 0"/>
+                <inertia
+                    ixx="0.1" ixy="0" ixz="0"
+                    iyy="0.1" iyz="0"
+                    izz="0.1"
+                />
+            </inertial>
+            <collision name='wheel_collision_${number}'>
+                <origin xyz="0 0 0" rpy="0 0 0"/>
+                <geometry>
+                    <cylinder radius="0.03" length="0.03"/>
+                </geometry>
+            </collision>
+            <visual name='wheel_visual_${number}'>
+                <origin xyz="0 0 0" rpy="0 0 0"/>
+                <geometry>
+                    <!-- <mesh filename="$(find tolya_description)/meshes/wheel.stl"/> -->
+                    <cylinder radius="0.03" length="0.03"/>
+                </geometry>
+            </visual>
         </link>
-        <joint name="wheel_joint_${number}" type="continuous">
+        <joint name="wheel_joint_${number}" type="fixed">
             <origin rpy="0 ${pi/2} 0" xyz="${origin_xyz}" />
             <parent link="${parent}" />
             <child link="wheel_link_${number}" />
-            <axis xyz="1 1 1" />
         </joint>
-    </xacro:macro >
+    </xacro:macro>
 </robot>
