Commit message: закоммитил хуету

File: simulation/workspace/src/tolya_description/urdf/base.xacro (robot description, xacro)
@@ -12,5 +12,5 @@
                 />
             </inertial>
-            <collision name='base_collision'>
+            <collision>
                 <origin xyz="0 0 0.06" rpy="0 0 0"/>
                 <geometry>
@@ -18,5 +18,5 @@
                 </geometry>
             </collision>
-            <visual name='base_visual'>
+            <visual>
                 <origin xyz="0 0 0.06" rpy="0 0 0"/>
                 <!-- <origin xyz="-0.187 0 0" rpy="0 0 ${pi}"/> -->
@@ -28,28 +28,7 @@
         </link>
         <link name="base_footprint">
-            <visual name="base_footprint_visual">
-                <origin xyz="0 0 0" rpy="0 0 0" />
-                <geometry>
-                    <box size="0.001 0.001 0.001" />
-                </geometry>
-            </visual>
-            <inertial>
-                <mass value="0.05"/>
-                <origin xyz="0.0 0 0" rpy=" 0 0 0"/>
-                <inertia
-                    ixx="0" ixy="0" ixz="0"
-                    iyy="0" iyz="0"
-                    izz="0"
-                />
-            </inertial>
-            <collision name='base_footprint_collision'>
-                <origin xyz="0 0 0" rpy="0 0 0"/>
-                <geometry>
-                    <box size="0.001 0.001 0.001" />
-                </geometry>
-            </collision>
         </link>
         <joint name="base_link_joint" type="fixed">
-            <origin xyz="0 0 0" rpy="0 0 0" />
+            <origin xyz="0 0 0.06" rpy="0 0 0" />
             <parent link="base_footprint"/>
             <child link="base_link" />

File: simulation/workspace/src/tolya_description/urdf/sensors.xacro (robot description, xacro)
@@ -3,7 +3,9 @@
     <xacro:include filename="sensors/imu.xacro" />
     <xacro:include filename="sensors/camera.xacro" />
+    <xacro:include filename="sensors/lidar.xacro" />
     <xacro:macro name="sensors" params="parent">
         <xacro:imu_sensor parent="${parent}"/>
         <xacro:camera_sensor parent="${parent}"/>
+        <xacro:lidar_sensor parent="${parent}"/>
     </xacro:macro>
 </robot>

File: simulation/workspace/src/tolya_description/urdf/sensors/camera.xacro (robot description, xacro)
@@ -2,5 +2,5 @@
 <robot xmlns:xacro="http://www.ros.org/wiki/xacro">
     <xacro:macro name="camera_sensor" params="parent">
-        <link name="camera_frame">
+        <link name="camera_link">
             <collision>
                 <origin xyz="0 0 0" rpy="0 0 0"/>
@@ -24,7 +24,22 @@
             <origin xyz="0.15 0.0 0.1" rpy="0 0 0"/>
             <parent link="${parent}"/>
+            <child link="camera_link"/>
+        </joint>
+        <link name="camera_frame">
+        </link>
+        <joint name="camera_frame_joint" type="fixed">
+            <origin xyz="0 0 0" rpy="${-pi/2} 0 ${-pi/2}"/>
+            <parent link="camera_link"/>
             <child link="camera_frame"/>
         </joint>
-        <gazebo reference="camera_frame">
+<!--
+        <link name="cube">
+        </link>
+        <joint name="cube_frame_joint" type="fixed">
+            <origin xyz="0 0 0" rpy="0 0 0"/>
+            <parent link="camera_frame"/>
+            <child link="cube"/>
+        </joint> -->
+        <gazebo reference="camera_link">
             <sensor type="camera" name="camera">
                 <visualize>true</visualize>

File: simulation/workspace/src/tolya_description/urdf/sensors/imu.xacro (robot description, xacro)
@@ -17,4 +17,5 @@
                     <rpyOffset>0 0 0</rpyOffset>
                     <frameName>imu_link</frameName>
+                    <frameId>base_link</frameId>
                 </plugin>
                 <pose>0 0 0 0 0 0</pose>

File: simulation/workspace/src/tolya_description/urdf/tolya.urdf (robot description, URDF)
Before this commit: robot tolya, 7 links, 6 joints
Links:
- added link camera_link, mass 1e-5; collision box size=0.01 0.01 0.01; visual box size=0.01 0.01 0.01
- added link lidar, mass 1e-5; collision sphere ; visual sphere 
- link base_footprint: mass 0.05 -> None; geometry 
- link camera_frame: mass 1e-5 -> None; geometry 
Joints:
- added joint camera_frame_joint: type fixed, parent camera_link, child camera_frame, origin xyz=0 0 0 rpy=-1.5707963267948966 0 -1.5707963267948966
- added joint lidar_joint: type fixed, parent base_link, child lidar, origin xyz=0 0 0.17 rpy=0 0 0
- joint base_link_joint: origin xyz=0 0 0 rpy=0 0 0 -> xyz=0 0 0.06 rpy=0 0 0
- joint camera_joint: child camera_frame -> camera_link
