Commit message: Ура локализация работает (а навигация нет)

File: workspace/src/tolya/urdf/base.xacro (robot description, xacro)
@@ -30,5 +30,5 @@
         </link>
         <joint name="base_link_joint" type="fixed">
-            <origin xyz="0 0 0.06" rpy="0 0 0" />
+            <origin xyz="0 0 0" rpy="0 0 0" />
             <parent link="base_footprint"/>
             <child link="base_link" />

File: workspace/src/tolya/urdf/sensors/lidar.xacro (robot description, xacro)
@@ -6,7 +6,5 @@
                 <origin xyz="0 0 0" rpy="0 0 0" />
                 <geometry>
-                    <sphere>
-                        <radius>0.02</radius>
-                    </sphere>
+                    <sphere radius="0.01"/>
                 </geometry>
             </visual>
@@ -14,7 +12,5 @@
                 <origin xyz="0 0 0" rpy="0 0 0" />
                 <geometry>
-                    <sphere>
-                        <radius>0.02</radius>
-                    </sphere>
+                    <sphere radius="0.01"/>
                 </geometry>
             </collision>

File: workspace/src/tolya/urdf/tolya.urdf (robot description, URDF)
Before this commit: robot tolya, 9 links, 8 joints
Links:
- link lidar: geometry collision sphere radius=0.01; visual sphere radius=0.01
Joints:
- joint base_link_joint: origin xyz=0 0 0.06 rpy=0 0 0 -> xyz=0 0 0 rpy=0 0 0
