Commit message: Куча всего в том числе яндекс карты

File: workspace/src/tolya/urdf/tolya.urdf (robot description, URDF)
Before this commit: robot tolya, 9 links, 8 joints
Links:
- added link base_grip, mass 1e-5; collision box size=0.2 0.05 0.05; visual box size=0.2 0.1 0.05
- added link finger_left_grip, mass 1e-5; collision box size=0.1 0.02 0.05; visual box size=0.1 0.02 0.05
- added link finger_right_grip, mass 1e-5; collision box size=0.1 0.02 0.05; visual box size=0.1 0.02 0.05
Joints:
- added joint base_grip_joint: type prismatic, parent base_link, child base_grip, origin xyz=0.06 0.0 0.07 rpy=0 0 0, axis 1 0 0, limit lower=0 upper=0.1 effort=1000.0 velocity=0.5
- added joint finger_left_joint: type revolute, parent base_grip, child finger_left_grip, origin xyz=0.1 0.03 0.0 rpy=0 0 0, axis 0 0 1, limit lower=0 upper=1.57 effort=1000.0 velocity=0.5
- added joint finger_right_joint: type revolute, parent base_grip, child finger_right_grip, origin xyz=0.1 -0.03 0.0 rpy=0 0 0, axis 0 0 1, limit lower=-1.57 upper=0 effort=1000.0 velocity=0.5

File: workspace/src/tolya/urdf/tolya.xacro (robot description, xacro)
@@ -4,5 +4,7 @@
   <xacro:include filename="wheel.xacro" />
   <xacro:include filename="sensors.xacro" />
+  <xacro:include filename="grip.xacro" />
   <xacro:base/>
+  <xacro:grip parent="base_link"/>
   <xacro:wheel parent="base_link" origin_xyz="0.065 0.059 0.03" number="1"/>
   <xacro:wheel parent="base_link" origin_xyz="-0.065 -0.059 0.03" number="2"/>
